File: AlarmSystem.sch (EAGLE design)
At the start: 8 parts, among them U1 ARDUINOR3-DIMENSION, U2 HC_05, X1 HD44780LCD-1602

Commit message: Updated AlarmSystem.sch
Parts:
- removed U2: HC_05, Bluetooth_HC_05:HC_05
- added U$2: SD_CARD_MODULE, Lab2:SD_CARD_MODULE
- added U$3: HC_05_BLUETOOTH_MODULE, Lab2:HC_05_BLUETOOTH_MODULE
Connections:
- new net 5V: IO/EXPANDERPWR.VCC, PIR1.VDD, U$2.VCC, U$3.VCC, U1.5V
- new net GND: IO/EXPANDERPWR.GND, PIR1.GND, S1.3, SP1.-, U$2.GND, U$3.GND, U1.GND1
- new net N$1: S1.1, U1.D2
- new net N$10: IO/EXPANDERIC$1.P2, U$1.C3
- new net N$11: IO/EXPANDERIC$1.P3, U$1.C4
- new net N$12: IO/EXPANDERIC$1.P4, U$1.R1
- new net N$13: IO/EXPANDERIC$1.SCL, U1.SCL
- new net N$14: IO/EXPANDERIC$1.P5, U$1.R2
- new net N$15: IO/EXPANDERIC$1.P6, U$1.R3
- new net N$16: IO/EXPANDERIC$1.P7, U$1.R4
- new net N$17: IO/EXPANDERIC$1.SDA, U1.SDA
- new net N$18: U$3.RXD, U1.D7
- new net N$19: U$3.TXD, U1.D6
- new net N$2: PIR1.OUT, U1.D5
- new net N$3: SP1.+, U1.D3
- new net N$4: IO/EXPANDERIC$1.P0, U$1.C1
- new net N$5: IO/EXPANDERIC$1.P1, U$1.C2
- new net N$6: U$2.SCK, U1.D13
- new net N$7: U$2.CS, U1.D10
- new net N$8: U$2.MISO, U1.D12
- new net N$9: U$2.MOSI, U1.D11
Other:
- moved on the sheet: IO/EXPANDERIC$1, PIR1, S1, SP1, U$1

Commit message: Updated code and electrical scheme
Parts:
- removed SP1: SPEAKER/AL60P, adafruit:SPEAKER/AL60P
- removed X1: HD44780LCD-1602, adafruit:HD44780LCD-1602
- added BUZZER: SPEAKER/AL60P, adafruit:SPEAKER/AL60P
- added I2C_LCD: I2C_LCD, Lab2:I2C_LCD
- added LCD_1602: HD44780LCD-1602, adafruit:HD44780LCD-1602
- renumbered S1 to BUTTON, U$1 to KEY_PAD, U$2 to MICRO_SD_MODULE, U$3 to HC-05_BLUETOOTH_MODULE
Connections:
- new net N$21: I2C_LCD.K, LCD_1602.K
- new net N$22: I2C_LCD.A, LCD_1602.A
- new net N$23: I2C_LCD.DB7, LCD_1602.DB7
- new net N$24: I2C_LCD.DB6, LCD_1602.DB6
- new net N$25: I2C_LCD.DB5, LCD_1602.DB5
- new net N$26: I2C_LCD.DB4, LCD_1602.DB4
- new net N$27: I2C_LCD.DB3, LCD_1602.DB3
- new net N$28: I2C_LCD.DB2, LCD_1602.DB2
- new net N$29: I2C_LCD.DB1, LCD_1602.DB1
- new net N$30: I2C_LCD.DB0, LCD_1602.DB0
- new net N$31: I2C_LCD.E, LCD_1602.E
- new net N$32: I2C_LCD.RW, LCD_1602.RW
- new net N$33: I2C_LCD.RS, LCD_1602.RS
- new net N$34: I2C_LCD.VD, LCD_1602.VO
- new net N$39: I2C_LCD.SCL, U1.A5/SCL
- new net N$40: I2C_LCD.SDA, U1.A4/SDA
- new net VDD: I2C_LCD.VDD, LCD_1602.VDD
- new net VSS: I2C_LCD.VSS, LCD_1602.VSS
- net 5V: now also I2C_LCD.VCC
- net GND: now also BUZZER.-, I2C_LCD.GND; no longer SP1.-
- net N$3: now also BUZZER.+; no longer SP1.+

Commit message: Updated code and scheme
Other:
- note added: "I2C for LCD module"
Changed lines of the file:
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@@
 <sheet>
 <plain>
+<text x="162.56" y="58.42" size="1.778" layer="91">I2C for LCD module</text>
 </plain>
 <instances>
